File: Eagle/Printer.sch (EAGLE design)
At the start: 3 parts, among them U1 DRV8824PWPR

Commit message: as
as
Connections:
- new net 3.3V: U$1.3V3
- new net 5V: U$1.5V
- new net GND: U$1.GND@38
Changed lines of the file:
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@@
 </busses>
 <nets>
+<net name="GND" class="0">
+<segment>
+<pinref part="U$1" gate="G$1" pin="GND@38"/>
+<wire x1="35.56" y1="12.7" x2="22.86" y2="12.7" width="0.1524" layer="91"/>
+<label x="22.86" y="12.7" size="1.778" layer="95"/>
+</segment>
+</net>
+<net name="3.3V" class="0">
+<segment>
+<pinref part="U$1" gate="G$1" pin="3V3"/>
+<wire x1="71.12" y1="12.7" x2="76.2" y2="12.7" width="0.1524" layer="91"/>
+<label x="76.2" y="12.7" size="1.778" layer="95"/>
+</segment>
+</net>
+<net name="5V" class="0">
+<segment>
+<pinref part="U$1" gate="G$1" pin="5V"/>
+<wire x1="71.12" y1="58.42" x2="78.74" y2="58.42" width="0.1524" layer="91"/>
+<label x="78.74" y="58.42" size="1.778" layer="95"/>
+</segment>
+</net>
 </nets>
 </sheet>

Commit message: awd
sad
Parts:
- removed U$2: TFT, tftdisplay:TFT
- added TFT_DISPLAY: TFT, tftdisplay:TFT
Connections:
- new net N$1: TFT_DISPLAY.DC, U$1.IO2
- new net N$2: TFT_DISPLAY.CS, U$1.IO4
- new net N$3: TFT_DISPLAY.RESET, U$1.IO15
- new net N$4: TFT_DISPLAY.SCK, TFT_DISPLAY.SD_SCK, U$1.IO18
- new net N$7: TFT_DISPLAY.SDI, TFT_DISPLAY.SD_MOSI, U$1.IO23
- new net N$9: TFT_DISPLAY.SD_CS, U$1.IO5
- new net TFT: TFT_DISPLAY.SD_MISO, U$1.IO19
- net 3.3V: now also TFT_DISPLAY.LED, TFT_DISPLAY.VCC
- net GND: now also TFT_DISPLAY.GND
Other:
- note added: ": Display"
Changed lines of the file:
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@@
 <parts>
 <part name="U$1" library="ESP32-DEVKITC" deviceset="ESP32DEVKITC" device=""/>
-<part name="U$2" library="tftdisplay" deviceset="TFT" device=""/>
+<part name="TFT_DISPLAY" library="tftdisplay" deviceset="TFT" device=""/>
 <part name="U1" library="Texas Instruments_By_element14_Batch_1" deviceset="DRV8824PWPR" device=""/>
 </parts>
@@
 <sheet>
 <plain>
+<text x="-33.02" y="22.86" size="1.778" layer="91">: Display</text>
 </plain>
 <instances>
@@
 <attribute name="NAME" x="48.26" y="8.89" size="1.27" layer="95" rot="R180"/>
 </instance>
-<instance part="U$2" gate="G$1" x="190.5" y="33.02" smashed="yes"/>
+<instance part="TFT_DISPLAY" gate="G$1" x="-78.74" y="48.26" smashed="yes" rot="MR0"/>
 <instance part="U1" gate="A" x="81.28" y="-35.56" smashed="yes">
 <attribute name="NAME" x="75.9206" y="-3.5814" size="2.0828" layer="95" ratio="10" rot="SR0"/>
@@
 <label x="22.86" y="12.7" size="1.778" layer="95"/>
 </segment>
+<segment>
+<pinref part="TFT_DISPLAY" gate="G$1" pin="GND"/>
+<wire x1="0" y1="33.02" x2="5.08" y2="33.02" width="0.1524" layer="91"/>
+<label x="0" y="33.02" size="1.778" layer="95"/>
+</segment>
 </net>
 <net name="3.3V" class="0">
@@
 <wire x1="71.12" y1="12.7" x2="76.2" y2="12.7" width="0.1524" layer="91"/>
 <label x="76.2" y="12.7" size="1.778" layer="95"/>
+</segment>
+<segment>
+<pinref part="TFT_DISPLAY" gate="G$1" pin="LED"/>
+<wire x1="0" y1="48.26" x2="5.08" y2="48.26" width="0.1524" layer="91"/>
+<label x="0" y="48.26" size="1.778" layer="95"/>
+</segment>
+<segment>
+<pinref part="TFT_DISPLAY" gate="G$1" pin="VCC"/>
+<wire x1="0" y1="30.48" x2="5.08" y2="30.48" width="0.1524" layer="91"/>
+<label x="0" y="30.48" size="1.778" layer="95"/>
 </segment>
 </net>
@@
 </segment>
 </net>
+<net name="N$1" class="0">
+<segment>
+<pinref part="TFT_DISPLAY" gate="G$1" pin="DC"/>
+<wire x1="0" y1="40.64" x2="17.78" y2="40.64" width="0.1524" layer="91"/>
+<pinref part="U$1" gate="G$1" pin="IO2"/>
+<wire x1="17.78" y1="40.64" x2="17.78" y2="48.26" width="0.1524" layer="91"/>
+<wire x1="17.78" y1="48.26" x2="35.56" y2="48.26" width="0.1524" layer="91"/>
+</segment>
+</net>
+<net name="N$2" class="0">
+<segment>
+<pinref part="U$1" gate="G$1" pin="IO4"/>
+<wire x1="35.56" y1="43.18" x2="25.4" y2="43.18" width="0.1524" layer="91"/>
+<wire x1="25.4" y1="43.18" x2="25.4" y2="35.56" width="0.1524" layer="91"/>
+<pinref part="TFT_DISPLAY" gate="G$1" pin="CS"/>
+<wire x1="25.4" y1="35.56" x2="0" y2="35.56" width="0.1524" layer="91"/>
+</segment>
+</net>
+<net name="N$3" class="0">
+<segment>
+<pinref part="TFT_DISPLAY" gate="G$1" pin="RESET"/>
+<wire x1="0" y1="38.1" x2="12.7" y2="38.1" width="0.1524" layer="91"/>
+<wire x1="12.7" y1="38.1" x2="12.7" y2="50.8" width="0.1524" layer="91"/>
+<pinref part="U$1" gate="G$1" pin="IO15"/>
+<wire x1="12.7" y1="50.8" x2="35.56" y2="50.8" width="0.1524" layer="91"/>
+</segment>
+</net>
+<net name="N$4" class="0">
+<segment>
+<pinref part="U$1" gate="G$1" pin="IO18"/>
+<wire x1="35.56" y1="33.02" x2="10.16" y2="33.02" width="0.1524" layer="91"/>
+<wire x1="10.16" y1="33.02" x2="10.16" y2="45.72" width="0.1524" layer="91"/>
+<pinref part="TFT_DISPLAY" gate="G$1" pin="SCK"/>
+<wire x1="10.16" y1="45.72" x2="0" y2="45.72" width="0.1524" layer="91"/>
+<pinref part="TFT_DISPLAY" gate="G$1" pin="SD_SCK"/>
+<wire x1="-76.2" y1="50.8" x2="-76.2" y2="71.12" width="0.1524" layer="91"/>
+<wire x1="-76.2" y1="71.12" x2="10.16" y2="71.12" width="0.1524" layer="91"/>
+<wire x1="10.16" y1="71.12" x2="10.16" y2="45.72" width="0.1524" layer="91"/>
+<junction x="10.16" y="45.72"/>
+</segment>
+</net>
+<net name="TFT" class="0">
+<segment>
+<pinref part="TFT_DISPLAY" gate="G$1" pin="SD_MISO"/>
+<wire x1="-76.2" y1="48.26" x2="-83.82" y2="48.26" width="0.1524" layer="91"/>
+<wire x1="-83.82" y1="48.26" x2="-83.82" y2="17.78" width="0.1524" layer="91"/>
+<wire x1="-83.82" y1="17.78" x2="5.08" y2="17.78" width="0.1524" layer="91"/>
+<wire x1="5.08" y1="17.78" x2="5.08" y2="27.94" width="0.1524" layer="91"/>
+<wire x1="5.08" y1="27.94" x2="25.4" y2="27.94" width="0.1524" layer="91"/>
+<pinref part="U$1" gate="G$1" pin="IO19"/>
+<wire x1="25.4" y1="27.94" x2="25.4" y2="30.48" width="0.1524" layer="91"/>
+<wire x1="25.4" y1="30.48" x2="35.56" y2="30.48" width="0.1524" layer="91"/>
+</segment>
+</net>
+<net name="N$7" class="0">
+<segment>
+<pinref part="TFT_DISPLAY" gate="G$1" pin="SDI"/>
+<wire x1="0" y1="43.18" x2="20.32" y2="43.18" width="0.1524" layer="91"/>
+<wire x1="20.32" y1="43.18" x2="20.32" y2="20.32" width="0.1524" layer="91"/>
+<pinref part="U$1" gate="G$1" pin="IO23"/>
+<wire x1="20.32" y1="20.32" x2="20.32" y2="15.24" width="0.1524" layer="91"/>
+<wire x1="20.32" y1="15.24" x2="35.56" y2="15.24" width="0.1524" layer="91"/>
+<pinref part="TFT_DISPLAY" gate="G$1" pin="SD_MOSI"/>
+<wire x1="-76.2" y1="45.72" x2="-81.28" y2="45.72" width="0.1524" layer="91"/>
+<wire x1="-81.28" y1="45.72" x2="-81.28" y2="20.32" width="0.1524" layer="91"/>
+<wire x1="-81.28" y1="20.32" x2="20.32" y2="20.32" width="0.1524" layer="91"/>
+<junction x="20.32" y="20.32"/>
+</segment>
+</net>
+<net name="N$9" class="0">
+<segment>
+<pinref part="U$1" gate="G$1" pin="IO5"/>
+<wire x1="35.56" y1="35.56" x2="30.48" y2="35.56" width="0.1524" layer="91"/>
+<wire x1="30.48" y1="35.56" x2="30.48" y2="25.4" width="0.1524" layer="91"/>
+<wire x1="30.48" y1="25.4" x2="-76.2" y2="25.4" width="0.1524" layer="91"/>
+<pinref part="TFT_DISPLAY" gate="G$1" pin="SD_CS"/>
+<wire x1="-76.2" y1="25.4" x2="-76.2" y2="43.18" width="0.1524" layer="91"/>
+</segment>
+</net>

Commit message: asd
sad
Parts:
- removed U1: DRV8824PWPR, Texas Instruments_By_element14_Batch_1:DRV8824PWPR
- added LED, LED1, LED2, LED3: HLMP6, display-hp:HLMP6
- added MICROSWITCH, MICROSWITCH1, MICROSWITCH2, MICROSWITCH3: E3206S, relay:E3206S
- added MODSTAND, MODSTAND1, MODSTAND2, MODSTAND3: 150 ohm, rcl:R-US_0204/7
- added U$2, U$3, U$4: JOYSTICK, tftdisplay:JOYSTICK
- added U$5, U$6: HBRO, tftdisplay:HBRO
Connections:
- new net DATA: LED.K, LED1.K, LED2.K, LED3.K, MODSTAND.2, MODSTAND1.2, MODSTAND2.2, MODSTAND3.2
- new net N$10: LED3.A, MICROSWITCH32.S
- new net N$11: U$1.IO33, U$4.VRX
- new net N$12: U$1.IO32, U$4.VRY
- new net N$13: U$1.IO35, U$4.SW
- new net N$5: LED.A, MICROSWITCH2.S
- new net N$6: LED1.A, MICROSWITCH12.S
- new net N$8: LED2.A, MICROSWITCH22.S
- new net NULL: MICROSWITCH12.O, MICROSWITCH2.O, MICROSWITCH22.O, MICROSWITCH32.O
- new net VCC: MICROSWITCH12.P, MICROSWITCH2.P, MICROSWITCH22.P, MICROSWITCH32.P
- net 5V: now also U$4.5V
- net GND: now also MODSTAND.1, MODSTAND1.1, MODSTAND2.1, MODSTAND3.1, U$4.GND

Commit message: as
as
Connections:
- new net 12V: U$5.UMOT, U$6.UMOT
- new net N$14: U$1.IO25, U$5.STP
- new net N$15: U$1.IO26, U$5.DIR
- new net N$16: U$1.IO27, U$6.DIR
- new net N$17: U$1.IO14, U$6.STP
- net 5V: now also U$5.RST, U$5.SLP, U$6.RST, U$6.SLP
- net GND: now also U$5.GND, U$5.GND2, U$6.GND, U$6.GND2
Other:
- note added: "Hbro X-akse"
Changed lines of the file:
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@@
 <plain>
 <text x="-33.02" y="22.86" size="1.778" layer="91">: Display</text>
+<text x="15.24" y="-27.94" size="1.778" layer="91">Hbro X-akse</text>
 </plain>
 <instances>
@@
 <instance part="U$4" gate="G$1" x="134.62" y="53.34" smashed="yes"/>
 <instance part="U$5" gate="G$1" x="20.32" y="-30.48" smashed="yes" rot="R180"/>
-<instance part="U$6" gate="G$1" x="104.14" y="-30.48" smashed="yes" rot="R180"/>
+<instance part="U$6" gate="G$1" x="20.32" y="-63.5" smashed="yes" rot="R180"/>
 </instances>
 <busses>
@@
 <label x="106.68" y="55.88" size="1.778" layer="95"/>
 </segment>
+<segment>
+<pinref part="U$5" gate="G$1" pin="GND"/>
+<wire x1="33.02" y1="-38.1" x2="48.26" y2="-38.1" width="0.1524" layer="91"/>
+<label x="48.26" y="-38.1" size="1.778" layer="95"/>
+</segment>
+<segment>
+<pinref part="U$5" gate="G$1" pin="GND2"/>
+<wire x1="33.02" y1="-22.86" x2="48.26" y2="-22.86" width="0.1524" layer="91"/>
+<label x="48.26" y="-22.86" size="1.778" layer="95"/>
+</segment>
+<segment>
+<pinref part="U$6" gate="G$1" pin="GND"/>
+<wire x1="33.02" y1="-71.12" x2="48.26" y2="-71.12" width="0.1524" layer="91"/>
+<label x="48.26" y="-71.12" size="1.778" layer="95"/>
+</segment>
+<segment>
+<pinref part="U$6" gate="G$1" pin="GND2"/>
+<wire x1="33.02" y1="-55.88" x2="48.26" y2="-55.88" width="0.1524" layer="91"/>
+<label x="48.26" y="-55.88" size="1.778" layer="95"/>
+</segment>
 </net>
 <net name="3.3V" class="0">
@@
 <wire x1="121.92" y1="53.34" x2="106.68" y2="53.34" width="0.1524" layer="91"/>
 <label x="106.68" y="53.34" size="1.778" layer="95"/>
+</segment>
+<segment>
+<pinref part="U$5" gate="G$1" pin="SLP"/>
+<wire x1="12.7" y1="-33.02" x2="-5.08" y2="-33.02" width="0.1524" layer="91"/>
+<wire x1="-5.08" y1="-33.02" x2="-5.08" y2="-30.48" width="0.1524" layer="91"/>
+<pinref part="U$5" gate="G$1" pin="RST"/>
+<wire x1="12.7" y1="-30.48" x2="-5.08" y2="-30.48" width="0.1524" layer="91"/>
+<wire x1="-5.08" y1="-30.48" x2="-12.7" y2="-30.48" width="0.1524" layer="91"/>
+<junction x="-5.08" y="-30.48"/>
+<label x="-12.7" y="-30.48" size="1.778" layer="95"/>
+</segment>
+<segment>
+<pinref part="U$6" gate="G$1" pin="SLP"/>
+<wire x1="12.7" y1="-66.04" x2="-2.54" y2="-66.04" width="0.1524" layer="91"/>
+<wire x1="-2.54" y1="-66.04" x2="-2.54" y2="-63.5" width="0.1524" layer="91"/>
+<pinref part="U$6" gate="G$1" pin="RST"/>
+<wire x1="-2.54" y1="-63.5" x2="12.7" y2="-63.5" width="0.1524" layer="91"/>
+<wire x1="-2.54" y1="-63.5" x2="-7.62" y2="-63.5" width="0.1524" layer="91"/>
+<junction x="-2.54" y="-63.5"/>
+<label x="-7.62" y="-63.5" size="1.778" layer="95"/>
 </segment>
 </net>
@@
 </segment>
 </net>
+<net name="12V" class="0">
+<segment>
+<pinref part="U$5" gate="G$1" pin="UMOT"/>
+<wire x1="33.02" y1="-20.32" x2="48.26" y2="-20.32" width="0.1524" layer="91"/>
+<label x="48.26" y="-20.32" size="1.778" layer="95"/>
+</segment>
+<segment>
+<pinref part="U$6" gate="G$1" pin="UMOT"/>
+<wire x1="33.02" y1="-53.34" x2="48.26" y2="-53.34" width="0.1524" layer="91"/>
+<label x="48.26" y="-53.34" size="1.778" layer="95"/>
+</segment>
+</net>
+<net name="N$14" class="0">
+<segment>
+<pinref part="U$5" gate="G$1" pin="STP"/>
+<wire x1="12.7" y1="-35.56" x2="-17.78" y2="-35.56" width="0.1524" layer="91"/>
+<wire x1="-17.78" y1="-35.56" x2="-17.78" y2="0" width="0.1524" layer="91"/>
+<wire x1="-17.78" y1="0" x2="83.82" y2="0" width="0.1524" layer="91"/>
+<wire x1="83.82" y1="0" x2="83.82" y2="33.02" width="0.1524" layer="91"/>
+<pinref part="U$1" gate="G$1" pin="IO25"/>
+<wire x1="83.82" y1="33.02" x2="71.12" y2="33.02" width="0.1524" layer="91"/>
+</segment>
+</net>
+<net name="N$15" class="0">
+<segment>
+<pinref part="U$5" gate="G$1" pin="DIR"/>
+<wire x1="12.7" y1="-38.1" x2="-15.24" y2="-38.1" width="0.1524" layer="91"/>
+<wire x1="-15.24" y1="-38.1" x2="-15.24" y2="-2.54" width="0.1524" layer="91"/>
+<wire x1="-15.24" y1="-2.54" x2="86.36" y2="-2.54" width="0.1524" layer="91"/>
+<wire x1="86.36" y1="-2.54" x2="86.36" y2="35.56" width="0.1524" layer="91"/>
+<pinref part="U$1" gate="G$1" pin="IO26"/>
+<wire x1="86.36" y1="35.56" x2="71.12" y2="35.56" width="0.1524" layer="91"/>
+</segment>
+</net>
+<net name="N$16" class="0">
+<segment>
+<pinref part="U$1" gate="G$1" pin="IO27"/>
+<wire x1="71.12" y1="38.1" x2="88.9" y2="38.1" width="0.1524" layer="91"/>
+<wire x1="88.9" y1="38.1" x2="88.9" y2="-5.08" width="0.1524" layer="91"/>
+<wire x1="88.9" y1="-5.08" x2="-22.86" y2="-5.08" width="0.1524" layer="91"/>
+<wire x1="-22.86" y1="-5.08" x2="-22.86" y2="-71.12" width="0.1524" layer="91"/>
+<pinref part="U$6" gate="G$1" pin="DIR"/>
+<wire x1="-22.86" y1="-71.12" x2="12.7" y2="-71.12" width="0.1524" layer="91"/>
+</segment>
+</net>
+<net name="N$17" class="0">
+<segment>
+<pinref part="U$1" gate="G$1" pin="IO14"/>
+<wire x1="71.12" y1="40.64" x2="91.44" y2="40.64" width="0.1524" layer="91"/>
+<wire x1="91.44" y1="40.64" x2="91.44" y2="-7.62" width="0.1524" layer="91"/>
+<wire x1="91.44" y1="-7.62" x2="-20.32" y2="-7.62" width="0.1524" layer="91"/>
+<wire x1="-20.32" y1="-7.62" x2="-20.32" y2="-68.58" width="0.1524" layer="91"/>
+<pinref part="U$6" gate="G$1" pin="STP"/>
+<wire x1="-20.32" y1="-68.58" x2="12.7" y2="-68.58" width="0.1524" layer="91"/>
+</segment>
+</net>

Commit message: asd
sad
Parts:
- added M1: SERVO, SparkFun-Electromechanical:SERVO
- U$2, U$3: value JOYSTICK -> STEPPERMOTOR; device tftdisplay:JOYSTICK -> tftdisplay:STEPPERMOTOR
Connections:
- new net N$18: M1.SIG, U$1.IO12
- new net N$19: U$2.B2, U$5.2B
- new net N$20: U$2.B1, U$5.1B
- new net N$21: U$2.A1, U$5.1A
- new net N$22: U$2.A2, U$5.2A
- new net N$23: U$3.B2, U$6.2B
- new net N$24: U$3.B1, U$6.1B
- new net N$25: U$3.A1, U$6.1A
- new net N$26: U$3.A2, U$6.2A
- net 5V: now also M1.V+
- net DATA: now also U$1.IO0, U$1.IO13, U$1.IO16, U$1.IO34
- net GND: now also M1.GND
Other:
- note added: "Alarm system X1"
- note added: "Alarm system X2"
- note added: "Alarm system Y1"
- note added: "Alarm system Y2"
- note added: "Hbro Y-akse"
- note added: "Joystick"
- note added: "Steppermotor X-akse"
- note added: "Steppermotor Y-akse"
- moved on the sheet: LED, LED1, LED2, LED3, MICROSWITCH, MICROSWITCH1, MICROSWITCH2, MICROSWITCH3, MODSTAND, MODSTAND1, MODSTAND2, MODSTAND3

Commit message: asd
sad
Connections:
- removed net N$2: TFT_DISPLAY.CS, U$1.IO4
- removed net N$3 (its old number): TFT_DISPLAY.RESET, U$1.IO15
- new net N$1: TFT_DISPLAY.CS, U$1.IO15
- net N$9: now also TFT_DISPLAY.RESET
Changed lines of the file:
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@@
-</segment>
-</net>
-<net name="N$1" class="0">
-<segment>
-<pinref part="TFT_DISPLAY" gate="G$1" pin="DC"/>
-<wire x1="0" y1="40.64" x2="17.78" y2="40.64" width="0.1524" layer="91"/>
-<pinref part="U$1" gate="G$1" pin="IO2"/>
-<wire x1="17.78" y1="40.64" x2="17.78" y2="48.26" width="0.1524" layer="91"/>
-<wire x1="17.78" y1="48.26" x2="35.56" y2="48.26" width="0.1524" layer="91"/>
-</segment>
-</net>
-<net name="N$2" class="0">
-<segment>
-<pinref part="U$1" gate="G$1" pin="IO4"/>
-<wire x1="35.56" y1="43.18" x2="25.4" y2="43.18" width="0.1524" layer="91"/>
-<wire x1="25.4" y1="43.18" x2="25.4" y2="35.56" width="0.1524" layer="91"/>
-<pinref part="TFT_DISPLAY" gate="G$1" pin="CS"/>
-<wire x1="25.4" y1="35.56" x2="0" y2="35.56" width="0.1524" layer="91"/>
-</segment>
-</net>
-<net name="N$3" class="0">
-<segment>
-<pinref part="TFT_DISPLAY" gate="G$1" pin="RESET"/>
-<wire x1="0" y1="38.1" x2="12.7" y2="38.1" width="0.1524" layer="91"/>
-<wire x1="12.7" y1="38.1" x2="12.7" y2="50.8" width="0.1524" layer="91"/>
-<pinref part="U$1" gate="G$1" pin="IO15"/>
-<wire x1="12.7" y1="50.8" x2="35.56" y2="50.8" width="0.1524" layer="91"/>
 </segment>
 </net>
@@
 <segment>
 <pinref part="U$1" gate="G$1" pin="IO18"/>
-<wire x1="35.56" y1="33.02" x2="10.16" y2="33.02" width="0.1524" layer="91"/>
-<wire x1="10.16" y1="33.02" x2="10.16" y2="45.72" width="0.1524" layer="91"/>
-<pinref part="TFT_DISPLAY" gate="G$1" pin="SCK"/>
-<wire x1="10.16" y1="45.72" x2="0" y2="45.72" width="0.1524" layer="91"/>
+<wire x1="35.56" y1="33.02" x2="17.78" y2="33.02" width="0.1524" layer="91"/>
 <pinref part="TFT_DISPLAY" gate="G$1" pin="SD_SCK"/>
+<wire x1="17.78" y1="33.02" x2="10.16" y2="33.02" width="0.1524" layer="91"/>
 <wire x1="-76.2" y1="50.8" x2="-76.2" y2="71.12" width="0.1524" layer="91"/>
 <wire x1="-76.2" y1="71.12" x2="10.16" y2="71.12" width="0.1524" layer="91"/>
-<wire x1="10.16" y1="71.12" x2="10.16" y2="45.72" width="0.1524" layer="91"/>
-<junction x="10.16" y="45.72"/>
+<wire x1="10.16" y1="71.12" x2="10.16" y2="33.02" width="0.1524" layer="91"/>
+<pinref part="TFT_DISPLAY" gate="G$1" pin="SCK"/>
+<wire x1="0" y1="45.72" x2="17.78" y2="45.72" width="0.1524" layer="91"/>
+<wire x1="17.78" y1="45.72" x2="17.78" y2="33.02" width="0.1524" layer="91"/>
+<junction x="17.78" y="33.02"/>
 </segment>
 </net>
@@
 <net name="N$7" class="0">
 <segment>
-<pinref part="TFT_DISPLAY" gate="G$1" pin="SDI"/>
-<wire x1="0" y1="43.18" x2="20.32" y2="43.18" width="0.1524" layer="91"/>
-<wire x1="20.32" y1="43.18" x2="20.32" y2="20.32" width="0.1524" layer="91"/>
 <pinref part="U$1" gate="G$1" pin="IO23"/>
 <wire x1="20.32" y1="20.32" x2="20.32" y2="15.24" width="0.1524" layer="91"/>
@@
 <wire x1="-76.2" y1="45.72" x2="-81.28" y2="45.72" width="0.1524" layer="91"/>
 <wire x1="-81.28" y1="45.72" x2="-81.28" y2="20.32" width="0.1524" layer="91"/>
-<wire x1="-81.28" y1="20.32" x2="20.32" y2="20.32" width="0.1524" layer="91"/>
-<junction x="20.32" y="20.32"/>
+<wire x1="-81.28" y1="20.32" x2="7.62" y2="20.32" width="0.1524" layer="91"/>
+<pinref part="TFT_DISPLAY" gate="G$1" pin="SDI"/>
+<wire x1="7.62" y1="20.32" x2="20.32" y2="20.32" width="0.1524" layer="91"/>
+<wire x1="0" y1="43.18" x2="7.62" y2="43.18" width="0.1524" layer="91"/>
+<wire x1="7.62" y1="43.18" x2="7.62" y2="20.32" width="0.1524" layer="91"/>
+<junction x="7.62" y="20.32"/>
 </segment>
 </net>
@@
 <pinref part="TFT_DISPLAY" gate="G$1" pin="SD_CS"/>
 <wire x1="-76.2" y1="25.4" x2="-76.2" y2="43.18" width="0.1524" layer="91"/>
+<pinref part="TFT_DISPLAY" gate="G$1" pin="RESET"/>
+<wire x1="0" y1="38.1" x2="25.4" y2="38.1" width="0.1524" layer="91"/>
+<wire x1="25.4" y1="38.1" x2="25.4" y2="35.56" width="0.1524" layer="91"/>
+<wire x1="25.4" y1="35.56" x2="30.48" y2="35.56" width="0.1524" layer="91"/>
+<junction x="30.48" y="35.56"/>
 </segment>
 </net>
@@
 </segment>
 </net>
+<net name="N$1" class="0">
+<segment>
+<pinref part="TFT_DISPLAY" gate="G$1" pin="CS"/>
+<wire x1="0" y1="35.56" x2="22.86" y2="35.56" width="0.1524" layer="91"/>
+<wire x1="22.86" y1="35.56" x2="22.86" y2="50.8" width="0.1524" layer="91"/>
+<pinref part="U$1" gate="G$1" pin="IO15"/>
+<wire x1="22.86" y1="50.8" x2="35.56" y2="50.8" width="0.1524" layer="91"/>
+</segment>
+</net>
+<net name="N$3" class="0">
+<segment>
+<pinref part="TFT_DISPLAY" gate="G$1" pin="DC"/>
+<wire x1="0" y1="40.64" x2="20.32" y2="40.64" width="0.1524" layer="91"/>
+<wire x1="20.32" y1="40.64" x2="20.32" y2="48.26" width="0.1524" layer="91"/>
+<pinref part="U$1" gate="G$1" pin="IO2"/>
+<wire x1="20.32" y1="48.26" x2="35.56" y2="48.26" width="0.1524" layer="91"/>
+</segment>
+</net>
