File: Eagle/Printer.sch (EAGLE design)
At the start: 20 parts, among them M1 SERVO

Commit message: asaa
asas
Connections:
- new net N$2: TFT_DISPLAY.RESET, U$1.IO5
- net DATA: now also U$1.IO17; no longer U$1.IO0
- net N$11: now also U$1.IO25; no longer U$1.IO33
- net N$14: now also U$1.IO33; no longer U$1.IO25
- net N$9: now also U$1.IO4; no longer TFT_DISPLAY.RESET, U$1.IO5
Changed lines of the file:
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@@
 <net name="N$9" class="0">
 <segment>
-<pinref part="U$1" gate="G$1" pin="IO5"/>
-<wire x1="35.56" y1="35.56" x2="30.48" y2="35.56" width="0.1524" layer="91"/>
-<wire x1="30.48" y1="35.56" x2="30.48" y2="25.4" width="0.1524" layer="91"/>
 <wire x1="30.48" y1="25.4" x2="-76.2" y2="25.4" width="0.1524" layer="91"/>
 <pinref part="TFT_DISPLAY" gate="G$1" pin="SD_CS"/>
 <wire x1="-76.2" y1="25.4" x2="-76.2" y2="43.18" width="0.1524" layer="91"/>
-<pinref part="TFT_DISPLAY" gate="G$1" pin="RESET"/>
-<wire x1="0" y1="38.1" x2="25.4" y2="38.1" width="0.1524" layer="91"/>
-<wire x1="25.4" y1="38.1" x2="25.4" y2="35.56" width="0.1524" layer="91"/>
-<wire x1="25.4" y1="35.56" x2="30.48" y2="35.56" width="0.1524" layer="91"/>
-<junction x="30.48" y="35.56"/>
+<wire x1="30.48" y1="25.4" x2="30.48" y2="43.18" width="0.1524" layer="91"/>
+<pinref part="U$1" gate="G$1" pin="IO4"/>
+<wire x1="30.48" y1="43.18" x2="35.56" y2="43.18" width="0.1524" layer="91"/>
 </segment>
 </net>
@@
 <wire x1="-22.86" y1="99.06" x2="-22.86" y2="81.28" width="0.1524" layer="91"/>
 <wire x1="-22.86" y1="81.28" x2="25.4" y2="81.28" width="0.1524" layer="91"/>
-<pinref part="U$1" gate="G$1" pin="IO0"/>
-<wire x1="25.4" y1="45.72" x2="35.56" y2="45.72" width="0.1524" layer="91"/>
 <wire x1="25.4" y1="81.28" x2="25.4" y2="45.72" width="0.1524" layer="91"/>
+<wire x1="25.4" y1="45.72" x2="33.02" y2="45.72" width="0.1524" layer="91"/>
+<wire x1="33.02" y1="45.72" x2="33.02" y2="38.1" width="0.1524" layer="91"/>
+<pinref part="U$1" gate="G$1" pin="IO17"/>
+<wire x1="33.02" y1="38.1" x2="35.56" y2="38.1" width="0.1524" layer="91"/>
 </segment>
 <segment>
@@
 <pinref part="MODSTAND1" gate="G$1" pin="2"/>
 <junction x="22.86" y="109.22"/>
+<wire x1="27.94" y1="99.06" x2="27.94" y2="40.64" width="0.1524" layer="91"/>
 <pinref part="U$1" gate="G$1" pin="IO16"/>
-<wire x1="27.94" y1="99.06" x2="27.94" y2="40.64" width="0.1524" layer="91"/>
 <wire x1="27.94" y1="40.64" x2="35.56" y2="40.64" width="0.1524" layer="91"/>
 </segment>
@@
 <pinref part="U$4" gate="G$1" pin="VRX"/>
 <wire x1="121.92" y1="50.8" x2="93.98" y2="50.8" width="0.1524" layer="91"/>
-<wire x1="93.98" y1="50.8" x2="93.98" y2="30.48" width="0.1524" layer="91"/>
-<pinref part="U$1" gate="G$1" pin="IO33"/>
-<wire x1="93.98" y1="30.48" x2="71.12" y2="30.48" width="0.1524" layer="91"/>
+<wire x1="93.98" y1="50.8" x2="93.98" y2="33.02" width="0.1524" layer="91"/>
+<pinref part="U$1" gate="G$1" pin="IO25"/>
+<wire x1="93.98" y1="33.02" x2="71.12" y2="33.02" width="0.1524" layer="91"/>
 </segment>
 </net>
@@
 <wire x1="-17.78" y1="-35.56" x2="-17.78" y2="0" width="0.1524" layer="91"/>
 <wire x1="-17.78" y1="0" x2="83.82" y2="0" width="0.1524" layer="91"/>
-<wire x1="83.82" y1="0" x2="83.82" y2="33.02" width="0.1524" layer="91"/>
-<pinref part="U$1" gate="G$1" pin="IO25"/>
-<wire x1="83.82" y1="33.02" x2="71.12" y2="33.02" width="0.1524" layer="91"/>
+<wire x1="83.82" y1="0" x2="83.82" y2="30.48" width="0.1524" layer="91"/>
+<pinref part="U$1" gate="G$1" pin="IO33"/>
+<wire x1="83.82" y1="30.48" x2="71.12" y2="30.48" width="0.1524" layer="91"/>
 </segment>
 </net>
@@
 </segment>
 </net>
+<net name="N$2" class="0">
+<segment>
+<pinref part="U$1" gate="G$1" pin="IO5"/>
+<wire x1="25.4" y1="35.56" x2="35.56" y2="35.56" width="0.1524" layer="91"/>
+<wire x1="25.4" y1="38.1" x2="25.4" y2="35.56" width="0.1524" layer="91"/>
+<pinref part="TFT_DISPLAY" gate="G$1" pin="RESET"/>
+<wire x1="0" y1="38.1" x2="25.4" y2="38.1" width="0.1524" layer="91"/>
+</segment>
+</net>

Commit message: qsas
asd
as
Parts:
- added R1: 10k, SparkFun-Resistors:10KOHM-HORIZ-1/4W-1%
- added S5: (no value), SparkFun-Retired:TAC_SWITCHPTH
Connections:
- new net N$27: R1.2, S5.1
- net 3.3V: now also U$4.5V
- net 5V: now also S5.2; no longer U$4.5V
- net GND: now also R1.1
- net N$11: now also U$1.IO32; no longer U$1.IO25
- net N$12: now also U$1.IO25; no longer U$1.IO32
- net N$13: now also S5.3; no longer U$4.SW
Other:
- note added: "Alarm system X#"
- note added: "Alarm system X-"
- note added: "Alarm system Y#"
- note added: "Alarm system Y-"
- note removed: "Alarm system X1"
- note removed: "Alarm system X2"
- note removed: "Alarm system Y1"
- note removed: "Alarm system Y2"
Changed lines of the file:
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@@
 <layer number="56" name="wert" color="7" fill="1" visible="no" active="no"/>
 <layer number="57" name="tCAD" color="7" fill="1" visible="no" active="no"/>
+<layer number="58" name="bCopper" color="7" fill="1" visible="no" active="no"/>
 <layer number="59" name="tCarbon" color="7" fill="1" visible="no" active="no"/>
 <layer number="60" name="bCarbon" color="7" fill="1" visible="no" active="no"/>
@@
 <layer number="115" name="ReferenceISLANDS" color="7" fill="1" visible="no" active="no"/>
 <layer number="116" name="Patch_BOT" color="9" fill="4" visible="no" active="no"/>
+<layer number="117" name="PM_Ref" color="7" fill="1" visible="no" active="no"/>
 <layer number="118" name="Rect_Pads" color="7" fill="1" visible="no" active="no"/>
+<layer number="119" name="PF_Ref" color="7" fill="1" visible="no" active="no"/>
+<layer number="120" name="WFL_Ref" color="7" fill="1" visible="no" active="no"/>
 <layer number="121" name="_tsilk" color="7" fill="1" visible="no" active="no"/>
 <layer number="122" name="_bsilk" color="7" fill="1" visible="no" active="no"/>
@@
 <layer number="128" name="_bValues" color="7" fill="1" visible="no" active="no"/>
 <layer number="129" name="Mask" color="7" fill="1" visible="no" active="no"/>
+<layer number="130" name="SMDSTROOK" color="7" fill="1" visible="no" active="no"/>
 <layer number="131" name="tAdjust" color="7" fill="1" visible="no" active="no"/>
 <layer number="132" name="bAdjust" color="7" fill="1" visible="no" active="no"/>
+<layer number="133" name="bottom_silk" color="7" fill="1" visible="no" active="no"/>
+<layer number="134" name="silk_top" color="7" fill="1" visible="no" active="no"/>
+<layer number="135" name="silk_bottom" color="7" fill="1" visible="no" active="no"/>
+<layer number="136" name="silktop" color="7" fill="1" visible="no" active="no"/>
+<layer number="137" name="silkbottom" color="7" fill="1" visible="no" active="no"/>
+<layer number="138" name="EEE" color="7" fill="1" visible="no" active="no"/>
+<layer number="139" name="_tKeepout" color="7" fill="1" visible="no" active="no"/>
+<layer number="140" name="mbKeepout" color="7" fill="1" visible="no" active="no"/>
+<layer number="141" name="ASSEMBLY_TOP" color="7" fill="1" visible="no" active="no"/>
+<layer number="142" name="mbRestrict" color="7" fill="1" visible="no" active="no"/>
+<layer number="143" name="PLACE_BOUND_TOP" color="7" fill="1" visible="no" active="no"/>
 <layer number="144" name="Drill_legend" color="7" fill="1" visible="no" active="no"/>
+<layer number="145" name="DrillLegend_01-16" color="7" fill="1" visible="no" active="no"/>
+<layer number="146" name="DrillLegend_01-20" color="7" fill="1" visible="no" active="no"/>
+<layer number="147" name="PIN_NUMBER" color="7" fill="1" visible="no" active="no"/>
+<layer number="148" name="DrillLegend_01-20" color="7" fill="1" visible="no" active="no"/>
+<layer number="149" name="DrillLegend_02-15" color="7" fill="1" visible="no" active="no"/>
 <layer number="150" name="Notes" color="7" fill="1" visible="no" active="no"/>
 <layer number="151" name="HeatSink" color="7" fill="1" visible="no" active="no"/>
@@
 <layer number="154" name="FabDoc2" color="7" fill="1" visible="no" active="no"/>
 <layer number="155" name="FabDoc3" color="7" fill="1" visible="no" active="no"/>
+<layer number="166" name="AntennaArea" color="7" fill="1" visible="no" active="no"/>
+<layer number="168" name="4mmHeightArea" color="7" fill="1" visible="no" active="no"/>
+<layer number="191" name="mNets" color="7" fill="1" visible="no" active="no"/>
+<layer number="192" name="mBusses" color="7" fill="1" visible="no" active="no"/>
+<layer number="193" name="mPins" color="7" fill="1" visible="no" active="no"/>
+<layer number="194" name="mSymbols" color="7" fill="1" visible="no" active="no"/>
+<layer number="195" name="mNames" color="7" fill="1" visible="no" active="no"/>
+<layer number="196" name="mValues" color="7" fill="1" visible="no" active="no"/>
 <layer number="199" name="Contour" color="7" fill="1" visible="no" active="no"/>
 <layer number="200" name="200bmp" color="1" fill="10" visible="no" active="no"/>
@@
 <layer number="250" name="Descript" color="3" fill="1" visible="no" active="no"/>
 <layer number="251" name="SMDround" color="12" fill="11" visible="no" active="no"/>
+<layer number="253" name="Extra" color="7" fill="1" visible="no" active="no"/>
 <layer number="254" name="cooling" color="7" fill="1" visible="no" active="no"/>
 <layer number="255" name="routoute" color="7" fill="1" visible="no" active="no"/>
@@
 <part name="U$2" library="tftdisplay" deviceset="STEPPERMOTOR" device=""/>
 <part name="U$3" library="tftdisplay" deviceset="STEPPERMOTOR" device=""/>
+<part name="S5" library="SparkFun-Retired" deviceset="TAC_SWITCH" device="PTH">
+<attribute name="SPICEPREFIX" value="S"/>
+</part>
+<part name="R1" library="SparkFun-Resistors" deviceset="10KOHM" device="-HORIZ-1/4W-1%" value="10k"/>
 </parts>
 <sheets>
@@
 <text x="63.5" y="-33.02" size="1.778" layer="91">Steppermotor X-akse</text>
 <text x="132.08" y="55.88" size="1.778" layer="91">Joystick</text>
-<text x="-33.02" y="116.84" size="1.778" layer="91">Alarm system X1</text>
-<text x="27.94" y="116.84" size="1.778" layer="91">Alarm system X2</text>
-<text x="83.82" y="116.84" size="1.778" layer="91">Alarm system Y1</text>
-<text x="144.78" y="116.84" size="1.778" layer="91">Alarm system Y2</text>
+<text x="-33.02" y="116.84" size="1.778" layer="91">Alarm system X-</text>
+<text x="27.94" y="116.84" size="1.778" layer="91">Alarm system X#</text>
+<text x="83.82" y="116.84" size="1.778" layer="91">Alarm system Y-</text>
+<text x="144.78" y="116.84" size="1.778" layer="91">Alarm system Y#</text>
 </plain>
 <instances>
@@
 <instance part="U$2" gate="G$1" x="71.12" y="-27.94" smashed="yes"/>
 <instance part="U$3" gate="G$1" x="71.12" y="-60.96" smashed="yes"/>
+<instance part="S5" gate="S" x="137.16" y="27.94" smashed="yes" rot="R180">
+<attribute name="NAME" x="139.7" y="21.59" size="1.778" layer="95" rot="R180"/>
+<attribute name="VALUE" x="139.7" y="34.29" size="1.778" layer="96" rot="R180"/>
+</instance>
+<instance part="R1" gate="G$1" x="149.86" y="27.94" smashed="yes" rot="R180">
+<attribute name="NAME" x="149.86" y="26.416" size="1.778" layer="95" font="vector" rot="R180" align="bottom-center"/>
+<attribute name="VALUE" x="149.86" y="29.464" size="1.778" layer="96" font="vector" rot="R180" align="top-center"/>
+</instance>
 </instances>
 <busses>
@@
 <label x="104.14" y="-17.78" size="1.778" layer="95"/>
 </segment>
+<segment>
+<pinref part="R1" gate="G$1" pin="1"/>
+<wire x1="154.94" y1="27.94" x2="157.48" y2="27.94" width="0.1524" layer="91"/>
+<label x="157.48" y="27.94" size="1.778" layer="95" rot="R180"/>
+</segment>
 </net>
 <net name="3.3V" class="0">
@@
 <label x="0" y="30.48" size="1.778" layer="95"/>
 </segment>
+<segment>
+<pinref part="U$4" gate="G$1" pin="5V"/>
+<wire x1="121.92" y1="53.34" x2="106.68" y2="53.34" width="0.1524" layer="91"/>
+<label x="106.68" y="53.34" size="1.778" layer="95"/>
+</segment>
 </net>
 <net name="5V" class="0">
@@
 <wire x1="71.12" y1="58.42" x2="78.74" y2="58.42" width="0.1524" layer="91"/>
 <label x="78.74" y="58.42" size="1.778" layer="95"/>
-</segment>
-<segment>
-<pinref part="U$4" gate="G$1" pin="5V"/>
-<wire x1="121.92" y1="53.34" x2="106.68" y2="53.34" width="0.1524" layer="91"/>
-<label x="106.68" y="53.34" size="1.778" layer="95"/>
 </segment>
 <segment>
@@
 <wire x1="111.76" y1="-20.32" x2="104.14" y2="-20.32" width="0.1524" layer="91"/>
 <label x="104.14" y="-20.32" size="1.778" layer="95"/>
+</segment>
+<segment>
+<pinref part="S5" gate="S" pin="2"/>
+<wire x1="142.24" y1="30.48" x2="144.78" y2="30.48" width="0.1524" layer="91"/>
+<label x="144.78" y="30.48" size="1.778" layer="95" rot="R180"/>
 </segment>
 </net>
@@
 <pinref part="U$4" gate="G$1" pin="VRX"/>
 <wire x1="121.92" y1="50.8" x2="93.98" y2="50.8" width="0.1524" layer="91"/>
-<wire x1="93.98" y1="50.8" x2="93.98" y2="33.02" width="0.1524" layer="91"/>
-<pinref part="U$1" gate="G$1" pin="IO25"/>
-<wire x1="93.98" y1="33.02" x2="71.12" y2="33.02" width="0.1524" layer="91"/>
+<wire x1="93.98" y1="50.8" x2="93.98" y2="27.94" width="0.1524" layer="91"/>
+<pinref part="U$1" gate="G$1" pin="IO32"/>
+<wire x1="93.98" y1="27.94" x2="71.12" y2="27.94" width="0.1524" layer="91"/>
 </segment>
 </net>
@@
 <pinref part="U$4" gate="G$1" pin="VRY"/>
 <wire x1="121.92" y1="48.26" x2="96.52" y2="48.26" width="0.1524" layer="91"/>
-<wire x1="96.52" y1="48.26" x2="96.52" y2="27.94" width="0.1524" layer="91"/>
-<pinref part="U$1" gate="G$1" pin="IO32"/>
-<wire x1="96.52" y1="27.94" x2="71.12" y2="27.94" width="0.1524" layer="91"/>
-</segment>
-</net>
-<net name="N$13" class="0">
-<segment>
-<pinref part="U$4" gate="G$1" pin="SW"/>
-<wire x1="121.92" y1="45.72" x2="99.06" y2="45.72" width="0.1524" layer="91"/>
-<wire x1="99.06" y1="45.72" x2="99.06" y2="25.4" width="0.1524" layer="91"/>
-<pinref part="U$1" gate="G$1" pin="IO35"/>
-<wire x1="99.06" y1="25.4" x2="71.12" y2="25.4" width="0.1524" layer="91"/>
+<wire x1="96.52" y1="48.26" x2="96.52" y2="33.02" width="0.1524" layer="91"/>
+<pinref part="U$1" gate="G$1" pin="IO25"/>
+<wire x1="96.52" y1="33.02" x2="71.12" y2="33.02" width="0.1524" layer="91"/>
 </segment>
 </net>
@@
 </segment>
 </net>
+<net name="N$13" class="0">
+<segment>
+<pinref part="S5" gate="S" pin="3"/>
+<wire x1="132.08" y1="27.94" x2="106.68" y2="27.94" width="0.1524" layer="91"/>
+<wire x1="106.68" y1="27.94" x2="106.68" y2="25.4" width="0.1524" layer="91"/>
+<pinref part="U$1" gate="G$1" pin="IO35"/>
+<wire x1="106.68" y1="25.4" x2="71.12" y2="25.4" width="0.1524" layer="91"/>
+</segment>
+</net>
+<net name="N$27" class="0">
+<segment>
+<pinref part="R1" gate="G$1" pin="2"/>
+<pinref part="S5" gate="S" pin="1"/>
+<wire x1="144.78" y1="27.94" x2="142.24" y2="27.94" width="0.1524" layer="91"/>
+</segment>
+</net>
